File: pcb/pcb/DAC.sch (KiCad schematic (older format))
At the start: 25 parts

Commit message: Tidy up
Parts:
- C? (x12): symbol Device:C -> pcb-rescue:C-Device
- R? (x6): symbol Device:R -> pcb-rescue:R-Device
- U? (x3): symbol Amplifier_Operational:TL072 -> pcb-rescue:TL072-Amplifier_Operational
- U?: symbol Regulator_Linear:L78L12_SOT89 -> pcb-rescue:L78L12_SOT89-Regulator_Linear
- U?: symbol Regulator_Linear:L79L12_SOT89 -> pcb-rescue:L79L12_SOT89-Regulator_Linear
Changed lines of the file:
@@
 EESchema Schematic File Version 4
 LIBS:pcb-cache
-EELAYER 26 0
+EELAYER 30 0
 EELAYER END
 $Descr A4 11693 8268
@@
 	4000 3400 3850 3400
 $Comp
-L Device:C C?
+L pcb-rescue:C-Device C?
 U 1 1 5CB0C696
 P 3400 3400
@@
 $EndComp
 $Comp
-L Device:C C?
+L pcb-rescue:C-Device C?
 U 1 1 5CB0C6BE
 P 3100 3400
@@
 Connection ~ 3650 3550
 $Comp
-L Device:R R?
+L pcb-rescue:R-Device R?
 U 1 1 5CB0C9B7
 P 2400 2750
@@
 $EndComp
 $Comp
-L Device:C C?
+L pcb-rescue:C-Device C?
 U 1 1 5CB0CA1E
 P 2250 2900
@@
 $EndComp
 $Comp
-L Device:R R?
+L pcb-rescue:R-Device R?
 U 1 1 5CB0CB56
 P 2700 3100
@@
 $EndComp
 $Comp
-L Device:C C?
+L pcb-rescue:C-Device C?
 U 1 1 5CB0CBA8
 P 2550 3250
@@
 DAC_OUT_L
 $Comp
-L Device:C C?
+L pcb-rescue:C-Device C?
 U 1 1 5CB0D1C2
 P 3100 2700
@@
 $EndComp
 $Comp
-L Device:C C?
+L pcb-rescue:C-Device C?
 U 1 1 5CB0D208
 P 3100 2350
@@
 $EndComp
 $Comp
-L Device:C C?
+L pcb-rescue:C-Device C?
 U 1 1 5CB0D238
 P 3400 2350
@@
 Connection ~ 3400 2550
 $Comp
-L Device:C C?
+L pcb-rescue:C-Device C?
 U 1 1 5CB0E05A
 P 3650 2650
@@
 	3100 2900 4000 2900
 $Comp
-L Device:C C?
+L pcb-rescue:C-Device C?
 U 1 1 5CB0F338
 P 5450 2250
@@
 $EndComp
 $Comp
-L Device:C C?
+L pcb-rescue:C-Device C?
 U 1 1 5CB0F3AE
 P 5850 2250
@@
 $EndComp
 $Comp
-L Device:C C?
+L pcb-rescue:C-Device C?
 U 1 1 5CB0F3E4
 P 5450 2600
@@
 $EndComp
 $Comp
-L Device:C C?
+L pcb-rescue:C-Device C?
 U 1 1 5CB0F42C
 P 5850 2600
@@
 	5450 3300 5000 3300
 $Comp
-L Amplifier_Operational:TL072 U?
+L pcb-rescue:TL072-Amplifier_Operational U?
 U 1 1 5CB17A70
 P 5300 4450
@@
 $EndComp
 $Comp
-L Amplifier_Operational:TL072 U?
+L pcb-rescue:TL072-Amplifier_Operational U?
 U 2 1 5CB17B0F
 P 5300 5950
@@
 $EndComp
 $Comp
-L Amplifier_Operational:TL072 U?
+L pcb-rescue:TL072-Amplifier_Operational U?
 U 3 1 5CB17BAB
 P 6900 4450
@@
 DAC_OUT_L
 $Comp
-L Device:R R?
+L pcb-rescue:R-Device R?
 U 1 1 5CB17EF0
 P 5300 4850
@@
 $EndComp
 $Comp
-L Device:R R?
+L pcb-rescue:R-Device R?
 U 1 1 5CB17F86
 P 4850 5000
@@
 Connection ~ 5700 4450
 $Comp
-L Device:R R?
+L pcb-rescue:R-Device R?
 U 1 1 5CB1D896
 P 5300 6350
@@
 $EndComp
 $Comp
-L Device:R R?
+L pcb-rescue:R-Device R?
 U 1 1 5CB1D926
 P 4850 6500
@@
 OUT_R
 $Comp
-L Regulator_Linear:L78L12_SOT89 U?
+L pcb-rescue:L78L12_SOT89-Regulator_Linear U?
 U 1 1 5CB245C2
 P 7950 1550
@@
 $EndComp
 $Comp
-L Regulator_Linear:L79L12_SOT89 U?
+L pcb-rescue:L79L12_SOT89-Regulator_Linear U?
 U 1 1 5CB247DA
 P 7950 2550
