File: pcb/pcb/I2S Serial Expander.sch (KiCad schematic (older format))
At the start: 8 parts

Commit message: Tidy up
Parts:
- U? (x4): symbol 74xx:74HC595 -> pcb-rescue:74HC595-74xx
Changed lines of the file:
@@
 EESchema Schematic File Version 4
 LIBS:pcb-cache
-EELAYER 26 0
+EELAYER 30 0
 EELAYER END
 $Descr A4 11693 8268
@@
 $EndDescr
 $Comp
-L 74xx:74HC595 U?
+L pcb-rescue:74HC595-74xx U?
 U 1 1 5CAC3687
 P 1700 4700
+AR Path="/5CAC3687" Ref="U?"  Part="1"
+AR Path="/5CAC35BA/5CAC3687" Ref="U?"  Part="1"
 F 0 "U?" H 1300 5450 50  0000 C CNN
 F 1 "74HC595" H 1400 5350 50  0000 C CNN
@@
 	1300 4800 1100 4800
 $Comp
-L 74xx:74HC595 U?
+L pcb-rescue:74HC595-74xx U?
 U 1 1 5CAC376A
 P 3450 4700
+AR Path="/5CAC376A" Ref="U?"  Part="1"
+AR Path="/5CAC35BA/5CAC376A" Ref="U?"  Part="1"
 F 0 "U?" H 3050 5450 50  0000 C CNN
 F 1 "74HC595" H 3150 5350 50  0000 C CNN
@@
 $EndComp
 $Comp
-L 74xx:74HC595 U?
+L pcb-rescue:74HC595-74xx U?
 U 1 1 5CAC3794
 P 5300 4700
+AR Path="/5CAC3794" Ref="U?"  Part="1"
+AR Path="/5CAC35BA/5CAC3794" Ref="U?"  Part="1"
 F 0 "U?" H 4900 5450 50  0000 C CNN
 F 1 "74HC595" H 5000 5350 50  0000 C CNN
@@
 $EndComp
 $Comp
-L 74xx:74HC595 U?
+L pcb-rescue:74HC595-74xx U?
 U 1 1 5CAC37E2
 P 7200 4700
+AR Path="/5CAC37E2" Ref="U?"  Part="1"
+AR Path="/5CAC35BA/5CAC37E2" Ref="U?"  Part="1"
 F 0 "U?" H 6800 5450 50  0000 C CNN
 F 1 "74HC595" H 6900 5350 50  0000 C CNN
