File: pcb/pcb/pcb.sch (KiCad schematic (older format))
At the start: 21 parts

Commit message: Tidy up
Parts:
- C? (x7): symbol Device:C -> pcb-rescue:C-Device
- D?: symbol Device:LED -> pcb-rescue:LED-Device
- D?: symbol Device:D -> pcb-rescue:D-Device
- R? (x8): symbol Device:R -> pcb-rescue:R-Device
- U?: symbol ESP32-footprints-Shem-Lib:ESP32-WROOM -> pcb-rescue:ESP32-WROOM-ESP32-footprints-Shem-Lib
- U?: symbol Regulator_Linear:NCP1117-3.3_SOT223 -> pcb-rescue:NCP1117-3.3_SOT223-Regulator_Linear
Connections:
- wire segments 77 -> 78
Changed lines of the file:
@@
 EESchema Schematic File Version 4
 LIBS:pcb-cache
-EELAYER 26 0
+EELAYER 30 0
 EELAYER END
 $Descr A4 11693 8268
@@
 $EndDescr
 $Comp
-L ESP32-footprints-Shem-Lib:ESP32-WROOM U?
+L pcb-rescue:ESP32-WROOM-ESP32-footprints-Shem-Lib U?
 U 1 1 5CA8B052
 P 6700 2150
@@
 	7750 2800 7750 2700
 $Comp
-L Regulator_Linear:NCP1117-3.3_SOT223 U?
+L pcb-rescue:NCP1117-3.3_SOT223-Regulator_Linear U?
 U 1 1 5CA9D870
 P 2650 1550
@@
 $EndComp
 $Comp
-L Device:C C?
+L pcb-rescue:C-Device C?
 U 1 1 5CA9DB7C
 P 2100 1850
@@
 $EndComp
 $Comp
-L Device:C C?
+L pcb-rescue:C-Device C?
 U 1 1 5CA9DBE7
 P 3150 1800
@@
 $EndComp
 $Comp
-L Device:R R?
+L pcb-rescue:R-Device R?
 U 1 1 5CA9DC48
 P 1700 1800
@@
 $EndComp
 $Comp
-L Device:LED D?
+L pcb-rescue:LED-Device D?
 U 1 1 5CA9DCCE
 P 1700 2100
@@
 $EndComp
 $Comp
-L Device:C C?
+L pcb-rescue:C-Device C?
 U 1 1 5CA9E1B5
 P 4450 1700
@@
 $EndComp
 $Comp
-L Device:C C?
+L pcb-rescue:C-Device C?
 U 1 1 5CA9E1E3
 P 5050 1700
@@
 $EndComp
 $Comp
-L Device:R R?
+L pcb-rescue:R-Device R?
 U 1 1 5CA9EA2B
 P 1800 3600
@@
 $EndComp
 $Comp
-L Device:C C?
+L pcb-rescue:C-Device C?
 U 1 1 5CA9EA90
 P 1800 4050
@@
 $EndComp
 $Comp
-L Device:C C?
+L pcb-rescue:C-Device C?
 U 1 1 5CAA03BC
 P 1450 6200
@@
 $EndComp
 $Comp
-L Device:C C?
+L pcb-rescue:C-Device C?
 U 1 1 5CAA0420
 P 1100 6200
@@
 SD_CMD
 $Comp
-L Device:R R?
+L pcb-rescue:R-Device R?
 U 1 1 5CAA0FD7
 P 2600 5450
@@
 	2600 5800 1950 5800
 $Comp
-L Device:R R?
+L pcb-rescue:R-Device R?
 U 1 1 5CAA19B8
 P 2350 5450
@@
 Connection ~ 2350 5900
 $Comp
-L Device:R R?
+L pcb-rescue:R-Device R?
 U 1 1 5CAA261C
 P 2100 5450
@@
 Connection ~ 2100 6000
 $Comp
-L Device:R R?
+L pcb-rescue:R-Device R?
 U 1 1 5CAA3397
 P 2600 6700
@@
 $EndComp
 $Comp
-L Device:R R?
+L pcb-rescue:R-Device R?
 U 1 1 5CAA3415
 P 2350 6700
@@
 $EndComp
 $Comp
-L Device:R R?
+L pcb-rescue:R-Device R?
 U 1 1 5CAA344F
 P 2100 6700
@@
 $EndComp
 $Comp
-L Device:D D?
+L pcb-rescue:D-Device D?
 U 1 1 5CAC0372
 P 5600 6300
@@
 F1 "DAC.sch" 50
 $EndSheet
+$Comp
+L power:+3.3V #PWR?
+U 1 1 5E0AC552
+P 9150 4850
+F 0 "#PWR?" H 9150 4700 50  0001 C CNN
+F 1 "+3.3V" H 9165 5023 50  0000 C CNN
+F 2 "" H 9150 4850 50  0001 C CNN
+F 3 "" H 9150 4850 50  0001 C CNN
+	1    9150 4850
+	0    -1   -1   0
+$EndComp
+Wire Wire Line
+	9350 4850 9150 4850
 $EndSCHEMATC
